File: kicad/_autosave-christmas_board.kicad_pcb (KiCad board)
At the start: 2 copper layers, 93.7 x 129.4 mm, 22 parts, among them J1 Conn_01x08, J2 Conn_01x04, SW1 SW_Push, SW2 SW_Push, SW3 SW_Push, SW4 SW_Push, SW5 SW_Push, SW6 SW_Push, SW7 SW_Push, SW8 SW_Push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

Commit message: mkd logo rauf geklatscht klappt aber noch net
Parts:
- moved G*** 1.27 mm to (147.3, 125.7)
Changed lines of the file:
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@@
       (outputformat 1)
       (mirror false)
-      (drillshape 1)
+      (drillshape 0)
       (scaleselection 1)
       (outputdirectory ""))
@@
   )
   (module graphics:40sLogo (layer B.Cu)
-    (at 147.32 127 180)
+    (at 147.32 125.73 180)
     (fp_text reference G*** (at 0 0) (layer B.SilkS) hide
       (effects (font (size 1.524 1.524) (thickness 0.3)) (justify mirror))
