File: kicad/christmas_board.kicad_pcb (KiCad board)
At the start: 2 copper layers, 93.7 x 129.4 mm, 22 parts, among them J1 Conn_01x08, J2 Conn_01x04, SW1 SW_Push, SW2 SW_Push, SW3 SW_Push, SW4 SW_Push, SW5 SW_Push, SW6 SW_Push, SW7 SW_Push, SW8 SW_Push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

Commit message: fixed
Parts:
- added G***: LOGO, graphics:mkd_logo_silk, B.Cu at (125.0, 98.0)
- moved G*** 1.70 mm to (123.4, 88.4)
- moved G*** 1.27 mm to (147.3, 125.7)
